Commit message: mistakenly updated the wrong mapper yaml

File: description/robot_core.xacro (robot description, xacro)
@@ -23,5 +23,5 @@
         <origin xyz="0 0 0" rpy="0 0 0"/>
     </joint>
-    <link name="base_link">
+    <link name="base_footprint">
     </link>
     <!-- CHASSIS LINK -->

Commit message: changes for SLAM

File: description/robot_core.xacro (robot description, xacro)
@@ -53,6 +53,6 @@
     </gazebo>
     <!-- LEFT WHEEL LINK -->
-    <joint name="rear_left_wheel_joint" type="continuous">
-        <parent link="base_link"/>
+    <joint name="rear_left_wheel_joint" type="fixed">
+        <parent link="chassis"/>
         <child link="rear_left_wheel"/>
         <origin xyz="-0.2 0.2 0" rpy="-${pi/2} 0 0" />
@@ -81,6 +81,6 @@
     </gazebo>
     <!-- RIGHT WHEEL LINK -->
-    <joint name="rear_right_wheel_joint" type="continuous">
-        <parent link="base_link"/>
+    <joint name="rear_right_wheel_joint" type="fixed">
+        <parent link="chassis"/>
         <child link="rear_right_wheel"/>
         <origin xyz="-0.2 -0.2 0" rpy="${pi/2} 0 0" />
